Commit message: update SF_TRON1A ARXR5 arm gripper URDF and EE frame

File: IsaacLab_RFM/source/ext_loco/ext_loco/assets/SF_TRON1A_ARXR5ARM/assembly.urdf (robot description, URDF)
Before this commit: robot assembly, 26 links, 25 joints
Links:
- removed link assembly
- removed link assembly_DAS_Controller_V3_with_flange
- removed link assembly_DAS_Controller_V3_with_flange_link1
- removed link assembly_DAS_Controller_V3_with_flange_link2
- removed link assembly_DAS_Controller_V3_with_flange_link3
- removed link assembly_DAS_Controller_V3_with_flange_link4
- removed link assembly_DAS_Controller_V3_with_flange_link5
- removed link assembly_DAS_Controller_V3_with_flange_link6
- removed link base_link_arm
- added link base_link, mass 0.42272; collision mesh filename=models/meshes/L5_umi/arm/raw_meshes_ARM/base_link_arm.STL; visual mesh filename=models/meshes/L5_umi/arm/raw_meshes_ARM/base_link_arm.STL
- added link eef_link, mass 0.0
- link link1: mass 0.096804 -> 0.09728; geometry collision mesh filename=models/meshes/L5_umi/arm/raw_meshes_ARM/link1.STL; visual mesh filename=models/meshes/L5_umi/arm/raw_meshes_ARM/link1.STL
- link link2: mass 1.1988 -> 1.1477; geometry collision mesh filename=models/meshes/L5_umi/arm/raw_meshes_ARM/link2.STL; visual mesh filename=models/meshes/L5_umi/arm/raw_meshes_ARM/link2.STL
- link link3: mass 0.84082 -> 0.66; geometry collision mesh filename=models/meshes/L5_umi/arm/raw_meshes_ARM/link3.STL; visual mesh filename=models/meshes/L5_umi/arm/raw_meshes_ARM/link3.STL
- link link4: mass 0.12432 -> 0.11714; geometry collision mesh filename=models/meshes/L5_umi/arm/raw_meshes_ARM/link4.STL; visual mesh filename=models/meshes/L5_umi/arm/raw_meshes_ARM/link4.STL
- link link5: mass 0.63601 -> 0.6353; geometry collision mesh filename=models/meshes/L5_umi/arm/raw_meshes_ARM/link5.STL; visual mesh filename=models/meshes/L5_umi/arm/raw_meshes_ARM/link5.STL
- link link6: mass 0.0139887 -> 0.902; geometry collision mesh filename=models/meshes/DAS_Controller_v3_r5_end_adapter_flange.STL scale=0.001 0.001 0.001; collision mesh filename=models/meshes/L5_umi/umi/base_link.STL
Joints:
- removed joint arm_base_joint
- removed joint assembly_DAS_Controller_V3_with_flange_joint1
- removed joint assembly_DAS_Controller_V3_with_flange_joint2
- removed joint assembly_DAS_Controller_V3_with_flange_joint3
- removed joint assembly_DAS_Controller_V3_with_flange_joint4
- removed joint assembly_DAS_Controller_V3_with_flange_joint5
- removed joint assembly_DAS_Controller_V3_with_flange_joint6
- removed joint assembly_DAS_Controller_V3_with_flange_joint_Flange
- added joint gripper_fixed_joint: type fixed, parent link6, child eef_link, origin xyz=0.0999414 0.0000388 0.0767217 rpy=0 0.2618 0
- joint J1: limit lower=-3.14 upper=2.618 effort=30 velocity=5 -> lower=-10 upper=10 effort=100 velocity=1000; parent base_link_arm -> base_link
- joint J2: limit lower=-0.05 upper=3.5 effort=40 velocity=5 -> lower=-10 upper=10 effort=100 velocity=1000
- joint J3: limit lower=-0.1 upper=3.2 effort=30 velocity=5.5 -> lower=-10 upper=10 effort=100 velocity=1000; origin xyz=-0.264 0 0 rpy=-3.1416 0 0 -> xyz=-0.264 0 0 rpy=3.1416 0 0
- joint J4: limit lower=-1.6 upper=1.55 effort=15 velocity=5.5 -> lower=-10 upper=10 effort=100 velocity=1000; origin xyz=0.245 -0.00005 -0.06 rpy=0 0 0 -> xyz=0.245 0 -0.06 rpy=0 0 0
- joint J5: limit lower=-1.57 upper=1.57 effort=10 velocity=5 -> lower=-10 upper=10 effort=100 velocity=1000; origin xyz=0.073914 0.00005 -0.083391 rpy=0 0 0 -> xyz=0.06775 -5E-05 -0.0865 rpy=0 0 0
- joint J6: limit lower=-3.14 upper=3.14 effort=3 velocity=6.28 -> lower=-10 upper=10 effort=100 velocity=1000; origin xyz=0.025286 0 0.083391 rpy=3.1415927 0 0 -> xyz=0.02895 0 0.0865 rpy=3.1416 0 0
- joint tron1computer-assembly: child base_link_arm -> base_link

Commit message: update sf tron1 arm assets/config

File: IsaacLab_RFM/source/ext_loco/ext_loco/assets/SF_TRON1A_ARXR5ARM/assembly.urdf (robot description, URDF)
Before this commit: robot assembly, 19 links, 18 joints
Joints:
- joint J1: limit lower=-10 upper=10 effort=100 velocity=1000 -> lower=-3.14 upper=2.618 effort=30 velocity=5
- joint J2: limit lower=-10 upper=10 effort=100 velocity=1000 -> lower=-0.05 upper=3.50 effort=40 velocity=5
- joint J3: limit lower=-10 upper=10 effort=100 velocity=1000 -> lower=-0.1 upper=3.2 effort=30 velocity=5.5
- joint J4: limit lower=-10 upper=10 effort=100 velocity=1000 -> lower=-1.6 upper=1.55 effort=15 velocity=5.5
- joint J5: limit lower=-10 upper=10 effort=100 velocity=1000 -> lower=-1.57 upper=1.57 effort=10 velocity=5
- joint J6: limit lower=-10 upper=10 effort=100 velocity=1000 -> lower=-2 upper=2 effort=10 velocity=5

Commit message: Align EEF frames and improve command-play support

File: IsaacLab_RFM/source/ext_loco/ext_loco/assets/SF_TRON1A_ARXR5ARM/assembly.urdf (robot description, URDF)
Before this commit: robot assembly, 19 links, 18 joints
Links:
- link eef_link: mass 0.0 -> 0.000001
Joints:
- joint gripper_fixed_joint: origin xyz=0.0999414 0.0000388 0.0767217 rpy=0 0.2618 0 -> xyz=0.15 0 0 rpy=0 0 0
